Commit message: Bring Vishnu's changes

File: urdf/include/erc_setup.urdf.xacro (robot description, xacro)
@@ -28,5 +28,5 @@
   </link>
   <joint name="zed2_tilt_head_joint" type="fixed">
-    <origin xyz="0 0 0.1291" rpy="0 0.415911961 0"/> <!-- 23.83 degree tilt -->
+    <origin xyz="0 0 0.1291" rpy="0 0.4 0"/>
     <parent link="erc_setup_link"/>
     <child link="zed2_tilt_head_link"/>

File: urdf/leo.urdf_viz.xacro (robot description, xacro)
@@ -7,5 +7,5 @@
   <xacro:include filename="$(find leo_description)/urdf/include/leo.gazebo.xacro"/>
   <xacro:include filename="$(find leo_description)/urdf/include/erc_setup.urdf.xacro"/>
-  <xacro:if value="$(arg fixed)">
+  <xacro:value="$(arg fixed)">
     <link name="world"/>
     <joint name="fixed" type="fixed">
@@ -14,5 +14,5 @@
       <origin xyz="0.0 0.0 0"/>
     </joint>
-  </xacro:if>
+  </xacro>
   <!-- MACROS -->
   <xacro:macro name="rocker_link" params="name">
